File: ps1.sch (KiCad schematic (older format))
At the start: 35 parts, among them P1 CONN_01X03, P2 CONN_01X03, T1 115V: 36VCT, 4A, U1 LM7818ACT, U2 LM7918ACT

Commit message: Cleared annotations, cleaned up annotations, added history block, modified title block. Component values do not indicate design parameters, all should be considered TBD.
Parts:
- U?: renamed from U1; value LM7818ACT -> LM7815ACT
- renumbered C1 to C?, C2 to C?, C7 to C?, D1 to D?, F1 to F?, L1 to L?, P1 to P?, P2 to P?, T1 to T?, U2 to U?
Other:
- note added: "26 December 2016"
- note added: "Date"
- note added: "Description"
- note added: "Discharge Protection"
- note added: "Engineer"
- note added: "Filter Network"
- note added: "Initial pre-release version"
- note added: "Matthew Pare"
- note added: "Release History"
- note added: "Rev."
- note added: "a"
- note removed: "C1, C2 35V\nC3, C4 50V\nC5, C6 35V\nC7, C8 50V"
- note removed: "Discharge\nProtection"
- note removed: "Earth Ground \nto chassis"
- note removed: "Virtual\nGround"
