File: kicad/ps1.kicad_pcb (KiCad board)
At the start: 2 copper layers, 36 parts, among them P1 CONN_01X03, P2 CONN_01X02, P3 CONN_01X02, P4 CONN_02X06, P5 CONN_02X06, U1 LM7815ACT, U2 LM7918ACT

Commit message: Umm, it has been a while since I committed to something.
Parts:
- moved P4 218.0 mm to (50.8, 204.5), turned to 0 degrees
- moved P5 213.9 mm to (86.4, 204.5), turned to 0 degrees
- moved D7 207.9 mm to (35.6, 193.0), turned to 0 degrees
- moved D6 206.1 mm to (118.1, 194.3), turned to 180 degrees
- moved R7 205.3 mm to (41.9, 193.0), turned to 180 degrees
- moved R6 203.6 mm to (110.5, 194.3), turned to 0 degrees
- moved P3 196.0 mm to (74.9, 191.8), turned to 270 degrees
- moved P2 195.8 mm to (82.5, 191.8), turned to 270 degrees
- moved R9 190.7 mm to (73.7, 188.0), turned to 0 degrees
- moved R8 190.4 mm to (81.3, 188.0), turned to 0 degrees
- moved R1 189.7 mm to (23.7, -90.8), turned to 0 degrees
- moved C1 188.5 mm to (33.9, -98.9), turned to 180 degrees
- moved C11 182.1 mm to (48.3, 177.8), turned to 180 degrees
- moved C10 181.6 mm to (113.0, 177.8), turned to 180 degrees
- moved R4 178.3 mm to (90.2, 179.1), turned to 270 degrees
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Other:
- board outline added: 139.7 x 190.5 mm

Commit message: New case and new layout.
Parts:
- removed P3: CONN_01X02, Pin_Headers:Pin_Header_Straight_1x02
- removed P4, P5: CONN_02X06, Connectors_Molex:Molex_MiniFit-JR-5556-12A_2x06x4.20mm_Straight
- removed R4, R5: R, Resistors_ThroughHole:Resistor_Ceramic_Horizontal_L19mm-W8mm-H8mm-p25mm
- removed R8, R9: R, Resistors_SMD:R_0805_HandSoldering
- removed the REF** at (92.7, 141.0)
- removed the REF** at (52.1, 141.0)
- added REF**: MountingHole_3.2mm_M3_Pad_Via, Mounting_Holes:MountingHole_3.2mm_M3_Pad_Via, F.Cu at (20.3, 80.0)
- added REF**: MountingHole_3.2mm_M3_Pad_Via, Mounting_Holes:MountingHole_3.2mm_M3_Pad_Via, F.Cu at (163.2, 81.9)
- added REF**: MountingHole_3.2mm_M3_Pad_Via, Mounting_Holes:MountingHole_3.2mm_M3_Pad_Via, F.Cu at (127.2, 50.4)
- added REF**: MountingHole_3.2mm_M3_Pad_Via, Mounting_Holes:MountingHole_3.2mm_M3_Pad_Via, F.Cu at (163.3, 19.7)
- added REF**: MountingHole_3.2mm_M3_Pad_Via, Mounting_Holes:MountingHole_3.2mm_M3_Pad_Via, F.Cu at (20.3, 20.3)
- added REF**: Heatsink_Fischer_SK129-STS_42x25mm_2xDrill2.5mm, Heatsinks:Heatsink_Fischer_SK129-STS_42x25mm_2xDrill2.5mm, F.Cu at (93.0, 67.3)
- added REF**: Heatsink_Fischer_SK129-STS_42x25mm_2xDrill2.5mm, Heatsinks:Heatsink_Fischer_SK129-STS_42x25mm_2xDrill2.5mm, F.Cu at (49.9, 67.3)
- added REF**: MountingHole_3.2mm_M3_Pad_Via, Mounting_Holes:MountingHole_3.2mm_M3_Pad_Via, F.Cu at (71.7, 67.2)
- C10, C11: footprint Capacitors_ThroughHole:C_Radial_D22_L41_P10 -> Capacitors_ThroughHole:C_Radial_D6.3_L11.2_P2.5
- C9: footprint Capacitors_ThroughHole:C_Disc_D12_P7.75 -> Capacitors_ThroughHole:C_Disc_D7.5_P5
- D1: footprint Diode_Bridge_18.5x5.5 -> ps1:Diode_Bridge_18.5x5.5
- P2: value CONN_01X02 -> CONN_01X03; footprint Pin_Headers:Pin_Header_Straight_1x02 -> ps1:Molex_Mini-Fit_JR-5566-03x3x
- moved R1 212.2 mm to (149.2, 80.3), turned to 90 degrees
- moved C1 207.3 mm to (156.8, 67.9), turned to 270 degrees
- moved D6 155.8 mm to (19.1, 74.1), turned to 270 degrees
- moved R6 149.1 mm to (22.9, 73.7), turned to 270 degrees
- moved R7 143.5 mm to (22.9, 50.8), turned to 90 degrees
- moved D7 142.7 mm to (19.7, 51.2), turned to 90 degrees
- moved P2 139.1 mm to (19.7, 67.7), turned to 90 degrees
- moved C10 131.0 mm to (93.3, 48.3)
- moved C11 129.0 mm to (52.1, 48.9), turned to 0 degrees
- moved P1 105.7 mm to (161.3, 61.4), turned to 90 degrees
- moved D4 103.4 mm to (87.9, 61.0), turned to 0 degrees
- moved D5 101.6 mm to (45.1, 61.0), turned to 0 degrees
- moved C8 86.2 mm to (96.0, 75.2), turned to 270 degrees
- moved C9 81.6 mm to (52.9, 80.3), turned to 90 degrees
- moved D2 80.0 mm to (87.9, 55.9)
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Connections:
- P2 pad 1: Net-(P2-Pad1) -> /+15V
Routing:
- net Net-(C3-Pad2): track 0.00 -> 142.0 mm
- net Net-(C2-Pad1): track 0.00 -> 74.1 mm
- net /-18V: track 0.00 -> 27.4 mm
- net /+18V: track 0.00 -> 24.7 mm
- net /-15V: track 0.00 -> 12.3 mm
- net Net-(C1-Pad2): track 0.00 -> 8.51 mm
- net /+15V: track 0.00 -> 4.13 mm
- net (no net): track 0.00 -> 1.75 mm
- added copper zone on B.Cu, net /GND
Other:
- board size 139.7 x 190.5 mm -> 152.4 x 139.7 mm
- net class Default: clearance 0.2 -> 0.6096; trace_width 0.25 -> 2.54
- rule trace_clearance: 0.2 -> 0.6096
